Commit message: SA E

File: src/test_urdf/urdf/test_arm_1018_new_new.urdf (robot description, URDF)
Before this commit: robot test_arm_1018_new_new, 8 links, 7 joints
Joints:
- joint joint0: limit lower=-2 upper=2 effort=100 velocity=1 -> lower=-2 upper=2 effort=28.0 velocity=1.0
- joint joint1: limit lower=-0.9 upper=1.5 effort=100 velocity=1 -> lower=-0.9 upper=1.5 effort=28.0 velocity=1.0
- joint joint2: limit lower=-3.14 upper=0.9 effort=100 velocity=1 -> lower=-3.14 upper=0.9 effort=28.0 velocity=1.0
- joint joint3: limit lower=-2 upper=1.5 effort=100 velocity=1 -> lower=-2.0 upper=1.5 effort=28.0 velocity=1.0
- joint joint4_0: limit lower=0 upper=2 effort=100 velocity=1 -> lower=0.0 upper=2.0 effort=28.0 velocity=1.0
- joint joint4_1: limit lower=-2 upper=0 effort=100 velocity=1 -> lower=-2.0 upper=0.0 effort=28.0 velocity=1.0

Commit message: if_ok_kikk 是可行的

File: src/test_urdf/urdf/test_arm_1018_new_new.urdf (robot description, URDF)
Before this commit: robot test_arm_1018_new_new, 8 links, 7 joints
Links:
- link base_link: mass 0.170234591037879 -> None
- link link0: mass 0.0134533721751118 -> None
- link link1: mass 0.0120579589553567 -> None
- link link2: mass 0.0163235420272894 -> None
- link link3: mass 0.0247731137376588 -> None
- link link4_0: mass 0.0086970283014079 -> None
- link link4_1: mass 0.0137369834582284 -> None
- link link4_end: mass 0.00183903257492059 -> None

Commit message: save

File: src/test_urdf/urdf/test_arm_1018_new_new.urdf (robot description, URDF)
Before this commit: robot test_arm_1018_new_new, 8 links, 7 joints
Joints:
- joint joint0: limit lower=-2 upper=2 effort=28.0 velocity=1.0 -> lower=-2 upper=2 effort=28.0 velocity=10.0
- joint joint1: limit lower=-0.9 upper=1.5 effort=28.0 velocity=1.0 -> lower=-0.9 upper=1.5 effort=28.0 velocity=10.0
- joint joint2: limit lower=-3.14 upper=0.9 effort=28.0 velocity=1.0 -> lower=-3.14 upper=0.9 effort=28.0 velocity=10.0
- joint joint3: limit lower=-2.0 upper=1.5 effort=28.0 velocity=1.0 -> lower=-2.0 upper=1.5 effort=28.0 velocity=10.0
- joint joint4_0: limit lower=0.0 upper=2.0 effort=28.0 velocity=1.0 -> lower=0.0 upper=2.0 effort=28.0 velocity=10.0
- joint joint4_1: limit lower=-2.0 upper=0.0 effort=28.0 velocity=1.0 -> lower=-2.0 upper=0.0 effort=28.0 velocity=10.0
