Commit message: 比较卡

File: src/robot_5dof/robo_description/urdf/robot_description.urdf (robot description, URDF)
Before this commit: robot robo_description, 8 links, 7 joints
Links:
- link base_link: mass 0.3102 -> None; geometry collision mesh filename=package://robo_description/meshes/visual/base_link.STL; visual mesh filename=package://robo_description/meshes/visual/base_link.STL
- link hand_link: mass 0.015548 -> None; geometry collision mesh filename=package://robo_description/meshes/visual/hand_link.STL; visual mesh filename=package://robo_description/meshes/visual/hand_link.STL
- link left_link: mass 0.008697 -> None; geometry collision mesh filename=package://robo_description/meshes/visual/left_link.STL; visual mesh filename=package://robo_description/meshes/visual/left_link.STL
- link right_link: mass 0.0091663 -> None; geometry collision mesh filename=package://robo_description/meshes/visual/right_link.STL; visual mesh filename=package://robo_description/meshes/visual/right_link.STL
- link robot_link1: mass 0.014963 -> None; geometry collision mesh filename=package://robo_description/meshes/visual/robot_link1.STL; visual mesh filename=package://robo_description/meshes/visual/robot_link1.STL
- link robot_link2: mass 0.010238 -> None; geometry collision mesh filename=package://robo_description/meshes/visual/robot_link2.STL; visual mesh filename=package://robo_description/meshes/visual/robot_link2.STL
- link robot_link3: mass 0.027294 -> None; geometry collision mesh filename=package://robo_description/meshes/visual/robot_link3.STL; visual mesh filename=package://robo_description/meshes/visual/robot_link3.STL
- link robot_link4: mass 0.019954 -> None; geometry collision mesh filename=package://robo_description/meshes/visual/robot_link4.STL; visual mesh filename=package://robo_description/meshes/visual/robot_link4.STL
Joints:
- removed joint left_link
- added joint left_joint: type revolute, parent hand_link, child left_link, origin xyz=0.0105 0 -0.083439 rpy=1.5708 0 0, axis 0 0 1, limit lower=-3.1 upper=3.1 effort=30 velocity=50.000001
- joint hand_joint: limit lower=-3.1 upper=3.1 effort=30 velocity=50 -> lower=-3.1 upper=3.1 effort=30 velocity=50.000001; origin xyz=0.001325 0.0678 0 rpy=-1.5708 0 0 -> xyz=0.001325 -0.17024 0 rpy=1.5708 1.5708 0
- joint right_joint: limit lower=-3.1 upper=3.1 effort=30 velocity=50 -> lower=-3.1 upper=3.1 effort=30 velocity=50.000001; mimic (none) -> joint=left_joint; origin xyz=0 0.0115 0.019 rpy=1.5708 0 -1.5708 -> xyz=-0.0115 0 -0.083439 rpy=-1.5708 0 3.1416
- joint robot_joint1: limit lower=-3.1 upper=3.1 effort=30 velocity=50 -> lower=-3.1 upper=3.1 effort=30 velocity=50.000001; origin xyz=0.080093 4.1073E-05 0.05375 rpy=0 0 0 -> xyz=-4.10730256436539E-05 0.0800931563628078 0.0537499999998397 rpy=0 0 0
- joint robot_joint2: axis 0 0 -1 -> 0 0 1; limit lower=-3.1 upper=3.1 effort=30 velocity=50 -> lower=-3.1 upper=3.1 effort=30 velocity=50.000001; origin xyz=-0.00080355 -0.0002 0.017887 rpy=1.5705 0 -0.00053478 -> xyz=0.00019999999985654 -0.000803554524565649 0.0178874681170878 rpy=-1.57107697491636 0 1.5702615513509
- joint robot_joint3: axis 0 0 -1 -> 0 0 1; limit lower=-3.1 upper=3.1 effort=30 velocity=50 -> lower=-3.1 upper=3.1 effort=30 velocity=50.000001; origin xyz=-1.2835E-05 0.081406 2.2853E-05 rpy=0.00028065 0.00053478 0 -> xyz=-1.28346100440498E-05 -0.0814055936788621 -2.28531912174905E-05 rpy=0.000280648161581886 -0.000534775422932215 0
- joint robot_joint4: axis 0 0 -1 -> 0 0 1; limit lower=-3.1 upper=3.1 effort=30 velocity=50 -> lower=-3.1 upper=3.1 effort=30 velocity=50.000001; origin xyz=0 0.07335 -0.00045 rpy=0 0 0 -> xyz=0 -0.07335 0.00045 rpy=0 0 0

Commit message: 5dof 修改，缺夹爪控制器

File: src/robot_5dof/robo_description/urdf/robot_description.urdf (robot description, URDF)
Before this commit: robot robo_description, 8 links, 7 joints
Joints:
- joint hand_joint: limit lower=-3.1 upper=3.1 effort=30 velocity=50.000001 -> lower=-0.5 upper=3.1 effort=30 velocity=50.000001
- joint left_joint: limit lower=-3.1 upper=3.1 effort=30 velocity=50.000001 -> lower=-1.1 upper=0 effort=30 velocity=50.000001
- joint robot_joint1: limit lower=-3.1 upper=3.1 effort=30 velocity=50.000001 -> lower=-2.0 upper=2.0 effort=30 velocity=50.000001
- joint robot_joint2: limit lower=-3.1 upper=3.1 effort=30 velocity=50.000001 -> lower=-0.9 upper=1.5 effort=30 velocity=50.000001
- joint robot_joint3: limit lower=-3.1 upper=3.1 effort=30 velocity=50.000001 -> lower=-2.1 upper=2.1 effort=30 velocity=50.000001
- joint robot_joint4: limit lower=-3.1 upper=3.1 effort=30 velocity=50.000001 -> lower=-2 upper=1.5 effort=30 velocity=50.000001
