Commit message: new_urdf

File: src/robot_5dof/robo_description/urdf/robo_description.urdf (robot description, URDF)
Before this commit: robot robo_description, 8 links, 7 joints
Joints:
- joint left_joint: limit lower=-1.1 upper=0 effort=30 velocity=50 -> lower=-0.027 upper=0 effort=30 velocity=50
- joint right_joint: axis 0 0 -1 -> 0 0 1; type revolute -> prismatic

Commit message: save left_joint->grippers_joint

File: src/robot_5dof/robo_description/urdf/robo_description.urdf (robot description, URDF)
Before this commit: robot robo_description, 8 links, 7 joints
Joints:
- removed joint left_joint
- added joint grippers_joint: type prismatic, parent hand_link, child left_link, origin xyz=0.026464 0.013587 -0.013325 rpy=-1.5708 0 -1.5708, axis 0 0 1, limit lower=-0.027 upper=0 effort=30 velocity=50
- joint right_joint: mimic joint=left_joint -> joint=grippers_joint

File: src/robot_5dof/robo_moveit/config/robo_description.ros2_control.xacro (robot description, xacro)
@@ -43,8 +43,8 @@
                 <state_interface name="velocity"/>
             </joint>
-            <joint name="left_joint">
+            <joint name="grippers_joint">
                 <command_interface name="position"/>
                 <state_interface name="position">
-                  <param name="initial_value">${initial_positions['left_joint']}</param>
+                  <param name="initial_value">${initial_positions['grippers_joint']}</param>
                 </state_interface>
                 <state_interface name="velocity"/>
